File: Kicad/lr_40/lr_40.kicad_sch (KiCad schematic)
At the start: 27 parts, among them J1 Screw_Terminal_01x02, J3 USB_C_Receptacle_PowerOnly_6P, Q1 MMBT3904, SW1 SW_DIP_x01, SW2 SW_DIP_x01, SW3 SW_DIP_x01, U1 MCP1700x-300xxTT, U2 ATtiny85V-10P, U3 BQ21040

Commit message: Nuova versione pcb
Parts:
- SW3: footprint Button_Switch_THT:SW_CK_JS202011CQN_DPDT_Straight -> Connector_PinSocket_2.54mm:PinSocket_1x03_P2.54mm_Vertical
Connections:
- net VCC: now also SW3.1; no longer SW3.2
- net laser: now also SW3.2; no longer SW3.1
Other:
- moved on the sheet: SW3
Changed lines of the file:
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@@
     (pin "1")
     (instances
-      (project "laser_rifle"
+      (project "laser_rifle_40mm.kicad_pro"
         (path "/be349321-04c2-4eb2-9cdd-764ade6a9fb1"
           (reference "#PWR07") (unit 1)
@@
     (pin "1")
     (instances
-      (project "laser_rifle"
+      (project "laser_rifle_40mm.kicad_pro"
         (path "/be349321-04c2-4eb2-9cdd-764ade6a9fb1"
           (reference "#PWR05") (unit 1)
@@
     (pin "1")
     (instances
-      (project "laser_rifle"
+      (project "laser_rifle_40mm.kicad_pro"
         (path "/be349321-04c2-4eb2-9cdd-764ade6a9fb1"
           (reference "#PWR09") (unit 1)
@@
     (pin "2")
     (instances
-      (project "laser_rifle"
+      (project "laser_rifle_40mm.kicad_pro"
         (path "/be349321-04c2-4eb2-9cdd-764ade6a9fb1"
           (reference "BT2") (unit 1)
@@
     (pin "1")
     (instances
-      (project "laser_rifle"
+      (project "laser_rifle_40mm.kicad_pro"
         (path "/be349321-04c2-4eb2-9cdd-764ade6a9fb1"
           (reference "R3") (unit 1)
@@
     (pin "2")
     (instances
-      (project "laser_rifle"
+      (project "laser_rifle_40mm.kicad_pro"
         (path "/be349321-04c2-4eb2-9cdd-764ade6a9fb1"
           (reference "U1") (unit 1)
@@
     (pin "1")
     (instances
-      (project "laser_rifle"
+      (project "laser_rifle_40mm.kicad_pro"
         (path "/be349321-04c2-4eb2-9cdd-764ade6a9fb1"
           (reference "J1") (unit 1)
@@
     (pin "1")
     (instances
-      (project "laser_rifle"
+      (project "laser_rifle_40mm.kicad_pro"
         (path "/be349321-04c2-4eb2-9cdd-764ade6a9fb1"
           (reference "#PWR013") (unit 1)
@@
     (pin "2")
     (instances
-      (project "laser_rifle"
+      (project "laser_rifle_40mm.kicad_pro"
         (path "/be349321-04c2-4eb2-9cdd-764ade6a9fb1"
           (reference "R4") (unit 1)
@@
     (pin "3")
     (instances
-      (project "laser_rifle"
+      (project "laser_rifle_40mm.kicad_pro"
         (path "/be349321-04c2-4eb2-9cdd-764ade6a9fb1"
           (reference "U3") (unit 1)
@@
     (pin "1")
     (instances
-      (project "laser_rifle"
+      (project "laser_rifle_40mm.kicad_pro"
         (path "/be349321-04c2-4eb2-9cdd-764ade6a9fb1"
           (reference "SW1") (unit 1)
@@
     (pin "2")
     (instances
-      (project "laser_rifle"
+      (project "laser_rifle_40mm.kicad_pro"
         (path "/be349321-04c2-4eb2-9cdd-764ade6a9fb1"
           (reference "R6") (unit 1)
@@
     (pin "1")
     (instances
-      (project "laser_rifle"
+      (project "laser_rifle_40mm.kicad_pro"
         (path "/be349321-04c2-4eb2-9cdd-764ade6a9fb1"
           (reference "C6") (unit 1)
@@
     (pin "3")
     (instances
-      (project "laser_rifle"
+      (project "laser_rifle_40mm.kicad_pro"
         (path "/be349321-04c2-4eb2-9cdd-764ade6a9fb1"
           (reference "U2") (unit 1)
@@
     )
   )
-  (symbol (lib_id "Switch:SW_DIP_x01") (at 137.16 121.92 90) (unit 1)
+  (symbol (lib_id "Switch:SW_DIP_x01") (at 137.16 121.92 270) (unit 1)
     (in_bom yes) (on_board yes) (dnp no) (fields_autoplaced)
     (property "Reference" "SW3" (at 140.97 120.65 90)
-      (effects (font (size 1.27 1.27)) (justify right))
+      (effects (font (size 1.27 1.27)) (justify left))
     )
     (property "Value" "SW_DIP_x01" (at 140.97 123.19 90)
-      (effects (font (size 1.27 1.27)) (justify right))
-    )
-    (property "Footprint" "Button_Switch_THT:SW_CK_JS202011CQN_DPDT_Straight" (at 137.16 121.92 0)
+      (effects (font (size 1.27 1.27)) (justify left))
+    )
+    (property "Footprint" "Connector_PinSocket_2.54mm:PinSocket_1x03_P2.54mm_Vertical" (at 137.16 121.92 0)
       (effects (font (size 1.27 1.27)) hide)
     )
@@
     (pin "2")
     (instances
-      (project "laser_rifle"
+      (project "laser_rifle_40mm.kicad_pro"
         (path "/be349321-04c2-4eb2-9cdd-764ade6a9fb1"
           (reference "SW3") (unit 1)
@@
     (pin "1")
     (instances
-      (project "laser_rifle"
+      (project "laser_rifle_40mm.kicad_pro"
         (path "/be349321-04c2-4eb2-9cdd-764ade6a9fb1"
           (reference "#PWR010") (unit 1)
@@
     (pin "1")
     (instances
-      (project "laser_rifle"
+      (project "laser_rifle_40mm.kicad_pro"
         (path "/be349321-04c2-4eb2-9cdd-764ade6a9fb1"
           (reference "R8") (unit 1)
@@
     (pin "1")
     (instances
-      (project "laser_rifle"
+      (project "laser_rifle_40mm.kicad_pro"
         (path "/be349321-04c2-4eb2-9cdd-764ade6a9fb1"
           (reference "#PWR012") (unit 1)
@@
     (pin "1")
     (instances
-      (project "laser_rifle"
+      (project "laser_rifle_40mm.kicad_pro"
         (path "/be349321-04c2-4eb2-9cdd-764ade6a9fb1"
           (reference "#PWR08") (unit 1)
@@
     (pin "1")
     (instances
-      (project "laser_rifle"
+      (project "laser_rifle_40mm.kicad_pro"
         (path "/be349321-04c2-4eb2-9cdd-764ade6a9fb1"
           (reference "#PWR011") (unit 1)
@@
     (pin "1")
     (instances
-      (project "laser_rifle"
+      (project "laser_rifle_40mm.kicad_pro"
         (path "/be349321-04c2-4eb2-9cdd-764ade6a9fb1"
           (reference "C4") (unit 1)
@@
     (pin "1")
     (instances
-      (project "laser_rifle"
+      (project "laser_rifle_40mm.kicad_pro"
         (path "/be349321-04c2-4eb2-9cdd-764ade6a9fb1"
           (reference "#PWR04") (unit 1)
@@
     (pin "2")
     (instances
-      (project "laser_rifle"
+      (project "laser_rifle_40mm.kicad_pro"
         (path "/be349321-04c2-4eb2-9cdd-764ade6a9fb1"
           (reference "C3") (unit 1)
@@
     (pin "1")
     (instances
-      (project "laser_rifle"
+      (project "laser_rifle_40mm.kicad_pro"
         (path "/be349321-04c2-4eb2-9cdd-764ade6a9fb1"
           (reference "Q1") (unit 1)
@@
     (pin "1")
     (instances
-      (project "laser_rifle"
+      (project "laser_rifle_40mm.kicad_pro"
         (path "/be349321-04c2-4eb2-9cdd-764ade6a9fb1"
           (reference "#PWR01") (unit 1)
@@
     (pin "1")
     (instances
-      (project "laser_rifle"
+      (project "laser_rifle_40mm.kicad_pro"
         (path "/be349321-04c2-4eb2-9cdd-764ade6a9fb1"
           (reference "D1") (unit 1)
@@
     (pin "1")
     (instances
-      (project "laser_rifle"
+      (project "laser_rifle_40mm.kicad_pro"
         (path "/be349321-04c2-4eb2-9cdd-764ade6a9fb1"
           (reference "D3") (unit 1)
@@
     (pin "1")
     (instances
-      (project "laser_rifle"
+      (project "laser_rifle_40mm.kicad_pro"
         (path "/be349321-04c2-4eb2-9cdd-764ade6a9fb1"
           (reference "#PWR02") (unit 1)
@@
     (pin "1")
     (instances
-      (project "laser_rifle"
+      (project "laser_rifle_40mm.kicad_pro"
         (path "/be349321-04c2-4eb2-9cdd-764ade6a9fb1"
           (reference "#PWR06") (unit 1)
@@
     (pin "1")
     (instances
-      (project "laser_rifle"
+      (project "laser_rifle_40mm.kicad_pro"
         (path "/be349321-04c2-4eb2-9cdd-764ade6a9fb1"
           (reference "C2") (unit 1)
@@
     (pin "1")
     (instances
-      (project "laser_rifle"
+      (project "laser_rifle_40mm.kicad_pro"
         (path "/be349321-04c2-4eb2-9cdd-764ade6a9fb1"
           (reference "R1") (unit 1)
@@
     (pin "2")
     (instances
-      (project "laser_rifle"
+      (project "laser_rifle_40mm.kicad_pro"
         (path "/be349321-04c2-4eb2-9cdd-764ade6a9fb1"
           (reference "R7") (unit 1)
@@
     (pin "1")
     (instances
-      (project "laser_rifle"
+      (project "laser_rifle_40mm.kicad_pro"
         (path "/be349321-04c2-4eb2-9cdd-764ade6a9fb1"
           (reference "D2") (unit 1)
@@
     (pin "1")
     (instances
-      (project "laser_rifle"
+      (project "laser_rifle_40mm.kicad_pro"
         (path "/be349321-04c2-4eb2-9cdd-764ade6a9fb1"
           (reference "C1") (unit 1)
@@
     (pin "1")
     (instances
-      (project "laser_rifle"
+      (project "laser_rifle_40mm.kicad_pro"
         (path "/be349321-04c2-4eb2-9cdd-764ade6a9fb1"
           (reference "#PWR03") (unit 1)
@@
     (pin "2")
     (instances
-      (project "laser_rifle"
+      (project "laser_rifle_40mm.kicad_pro"
         (path "/be349321-04c2-4eb2-9cdd-764ade6a9fb1"
           (reference "SW2") (unit 1)
@@
     (pin "2")
     (instances
-      (project "laser_rifle"
+      (project "laser_rifle_40mm.kicad_pro"
         (path "/be349321-04c2-4eb2-9cdd-764ade6a9fb1"
           (reference "R5") (unit 1)
@@
     (pin "1")
     (instances
-      (project "laser_rifle"
+      (project "laser_rifle_40mm.kicad_pro"
         (path "/be349321-04c2-4eb2-9cdd-764ade6a9fb1"
           (reference "R2") (unit 1)
@@
     (pin "A5")
     (instances
-      (project "laser_rifle"
+      (project "laser_rifle_40mm.kicad_pro"
         (path "/be349321-04c2-4eb2-9cdd-764ade6a9fb1"
           (reference "J3") (unit 1)
@@
     (pin "1")
     (instances
-      (project "laser_rifle"
+      (project "laser_rifle_40mm.kicad_pro"
         (path "/be349321-04c2-4eb2-9cdd-764ade6a9fb1"
           (reference "C7") (unit 1)
